File: vsource/vsource.kicad_sch (KiCad schematic)
At the start: 0 parts

Commit message: first commit
Parts:
- added C1, C2, C3, C4: C_US, symbol Device:C_US
- added D1, D2, D3, D4: 1N4007, Diode_THT:D_DO-41_SOD81_P10.16mm_Horizontal, symbol Diode:1N4007
- added J1, J2: Screw_Terminal_01x03, symbol Connector:Screw_Terminal_01x03
- added R1, R2: R_US, symbol Device:R_US
- added RV1, RV2: R_Potentiometer, symbol Device:R_Potentiometer
- added U1: LM317_TO-220, Package_TO_SOT_THT:TO-220-3_Vertical, symbol Regulator_Linear:LM317_TO-220
- added U2: LM337_TO220, Package_TO_SOT_THT:TO-220-3_Vertical, symbol Regulator_Linear:LM337_TO220
Connections:
- new net: D1.2 (A), D2.1 (K), J1.3 (Pin_3)
- new net: C2.2, D2.2 (A), D4.2 (A), U2.2 (VI)
- new net: R2.2, RV1.1, U1.1 (ADJ)
- new net: C1.2, C2.1, C3.2, C4.1, J1.2 (Pin_2), J2.2 (Pin_2), RV1.3, RV2.1
- new net: C1.1, D1.1 (K), D3.1 (K), U1.3 (VI)
- new net: D3.2 (A), D4.1 (K), J1.1 (Pin_1)
- new net: C4.2, J2.3 (Pin_3), R1.2, U2.3 (VO)
- new net: R1.1, RV2.3, U2.1 (ADJ)
- new net: C3.1, J2.1 (Pin_1), R2.1, U1.2 (VO)

Commit message: update
Parts:
- C1, C2: footprint (none) -> Capacitor_THT:CP_Radial_D16.0mm_P7.50mm
- C3, C4: footprint (none) -> Capacitor_THT:CP_Radial_D5.0mm_P2.50mm
- J1, J2: footprint (none) -> TerminalBlock_Altech:Altech_AK100_1x03_P5.00mm
- R1, R2: footprint (none) -> Resistor_THT:R_Axial_DIN0204_L3.6mm_D1.6mm_P7.62mm_Horizontal
- RV1, RV2: footprint (none) -> Potentiometer_THT:Potentiometer_Alps_RK09Y11_Single_Horizontal
Connections:
- net at RV1.2: now also C1.2, C2.1, C3.2, C4.1, J1.2 (Pin_2), J2.2 (Pin_2), RV1.3, RV2.1, RV2.2
- net at C4.2, J2.3 (Pin_3), U2.3 (VO): now also R1.1; no longer R1.2
- net at RV2.3, U2.1 (ADJ): now also R1.2; no longer R1.1
Other:
- moved on the sheet: R1
Changed lines of the file:
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@@
+	)
+	(junction
+		(at 110.49 71.12)
+		(diameter 0)
+		(color 0 0 0 0)
 	)
 	(junction
@@
 	)
 	(junction
+		(at 110.49 66.04)
+		(diameter 0)
+		(color 0 0 0 0)
+	)
+	(junction
 		(at 59.69 82.55)
 		(diameter 0)
@@
 	(wire
 		(pts
+			(xy 110.49 66.04) (xy 110.49 68.58)
+		)
+		(stroke
+			(width 0)
+			(type default)
+		)
+	)
+	(wire
+		(pts
+			(xy 123.19 95.25) (xy 133.35 95.25)
+		)
+		(stroke
+			(width 0)
+			(type default)
+		)
+	)
+	(wire
+		(pts
 			(xy 96.52 68.58) (xy 110.49 68.58)
 		)
@@
 	(wire
 		(pts
+			(xy 114.3 71.12) (xy 110.49 71.12)
+		)
+		(stroke
+			(width 0)
+			(type default)
+		)
+	)
+	(wire
+		(pts
 			(xy 121.92 46.99) (xy 133.35 46.99)
 		)
@@
 	(wire
 		(pts
+			(xy 114.3 60.96) (xy 114.3 66.04)
+		)
+		(stroke
+			(width 0)
+			(type default)
+		)
+	)
+	(wire
+		(pts
 			(xy 110.49 85.09) (xy 110.49 87.63)
 		)
@@
 	(wire
 		(pts
+			(xy 110.49 71.12) (xy 110.49 74.93)
+		)
+		(stroke
+			(width 0)
+			(type default)
+		)
+	)
+	(wire
+		(pts
 			(xy 102.87 95.25) (xy 96.52 95.25)
 		)
@@
 	(wire
 		(pts
-			(xy 110.49 64.77) (xy 110.49 68.58)
+			(xy 110.49 64.77) (xy 110.49 66.04)
 		)
 		(stroke
@@
 	(wire
 		(pts
-			(xy 123.19 95.25) (xy 133.35 95.25)
-		)
-		(stroke
-			(width 0)
-			(type default)
-		)
-	)
-	(wire
-		(pts
-			(xy 110.49 68.58) (xy 110.49 74.93)
+			(xy 114.3 66.04) (xy 110.49 66.04)
+		)
+		(stroke
+			(width 0)
+			(type default)
+		)
+	)
+	(wire
+		(pts
+			(xy 110.49 68.58) (xy 110.49 71.12)
 		)
 		(stroke
@@
 		(pts
 			(xy 96.52 91.44) (xy 96.52 95.25)
+		)
+		(stroke
+			(width 0)
+			(type default)
+		)
+	)
+	(wire
+		(pts
+			(xy 114.3 78.74) (xy 114.3 71.12)
 		)
 		(stroke
@@
 			)
 		)
-		(property "Footprint" ""
+		(property "Footprint" "Potentiometer_THT:Potentiometer_Alps_RK09Y11_Single_Horizontal"
 			(at 110.49 60.96 0)
 			(effects
@@
 			)
 		)
-		(property "Footprint" ""
+		(property "Footprint" "Capacitor_THT:CP_Radial_D5.0mm_P2.50mm"
 			(at 133.35 91.44 0)
 			(effects
@@
 			)
 		)
-		(property "Footprint" ""
+		(property "Footprint" "Potentiometer_THT:Potentiometer_Alps_RK09Y11_Single_Horizontal"
 			(at 110.49 78.74 0)
 			(effects
@@
 			)
 		)
-		(property "Footprint" ""
+		(property "Footprint" "TerminalBlock_Altech:Altech_AK100_1x03_P5.00mm"
 			(at 36.83 49.53 0)
 			(effects
@@
 			)
 		)
-		(property "Footprint" ""
+		(property "Footprint" "TerminalBlock_Altech:Altech_AK100_1x03_P5.00mm"
 			(at 153.67 49.53 0)
 			(effects
@@
 			)
 		)
-		(property "Footprint" ""
+		(property "Footprint" "Capacitor_THT:CP_Radial_D5.0mm_P2.50mm"
 			(at 133.35 50.8 0)
 			(effects
@@
 			)
 		)
-		(property "Footprint" ""
+		(property "Footprint" "Resistor_THT:R_Axial_DIN0204_L3.6mm_D1.6mm_P7.62mm_Horizontal"
 			(at 122.936 51.054 90)
 			(effects
@@
 			)
 		)
-		(property "Footprint" ""
+		(property "Footprint" "Capacitor_THT:CP_Radial_D16.0mm_P7.50mm"
 			(at 96.52 54.61 0)
 			(effects
@@
 	(symbol
 		(lib_id "Device:R_US")
-		(at 123.19 91.44 0)
+		(at 123.19 91.44 180)
 		(unit 1)
 		(exclude_from_sim no)
@@
 					(size 1.27 1.27)
 				)
-				(justify left)
+				(justify right)
 			)
 		)
@@
 					(size 1.27 1.27)
 				)
-				(justify left)
-			)
-		)
-		(property "Footprint" ""
-			(at 124.206 91.694 90)
+				(justify right)
+			)
+		)
+		(property "Footprint" "Resistor_THT:R_Axial_DIN0204_L3.6mm_D1.6mm_P7.62mm_Horizontal"
+			(at 122.174 91.186 90)
 			(effects
 				(font
@@
 			)
 		)
-		(property "Footprint" ""
+		(property "Footprint" "Capacitor_THT:CP_Radial_D16.0mm_P7.50mm"
 			(at 96.52 87.63 0)
 			(effects
